File: PCB Class/3.3V Regulator.kicad_sch (KiCad schematic)
At the start: 3 parts, among them U2 AP2112K-3.3TRG1

Commit message: Final Schematic
Connections:
- net VDD renamed +3.3V
Other:
- note removed: "Jan 10th 2024"
- note removed: "Riya Gupta LED Light Schematic"
- title: (none) -> RGB LED Lights
Changed lines of the file:
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@@
 (kicad_sch (version 20211123) (generator eeschema)
-  (paper "A4")
+  (paper "USLetter")
+  (title_block
+    (title "RGB LED Lights")
+    (date "2024-01-11")
+    (rev "B01")
+    (comment 1 "Riya Gupta")
+  )
   (junction (at 151.13 81.28) (diameter 0) (color 0 0 0 0)
+  )
+  (junction (at 154.94 71.12) (diameter 0) (color 0 0 0 0)
   )
   (junction (at 123.19 76.2) (diameter 0) (color 0 0 0 0)
@@
     (stroke (width 0) (type default) (color 0 0 0 0))
   )
+  (wire (pts (xy 154.94 71.12) (xy 157.48 71.12))
+    (stroke (width 0) (type default) (color 0 0 0 0))
+  )
   (wire (pts (xy 123.19 76.2) (xy 123.19 77.47))
     (stroke (width 0) (type default) (color 0 0 0 0))
   )
   (wire (pts (xy 125.73 76.2) (xy 123.19 76.2))
+    (stroke (width 0) (type default) (color 0 0 0 0))
+  )
+  (wire (pts (xy 154.94 68.58) (xy 154.94 71.12))
     (stroke (width 0) (type default) (color 0 0 0 0))
   )
@@
     (stroke (width 0) (type default) (color 0 0 0 0))
   )
-  (wire (pts (xy 151.13 71.12) (xy 157.48 71.12))
+  (wire (pts (xy 151.13 71.12) (xy 154.94 71.12))
     (stroke (width 0) (type default) (color 0 0 0 0))
   )
   (wire (pts (xy 151.13 71.12) (xy 151.13 73.66))
     (stroke (width 0) (type default) (color 0 0 0 0))
-  )
-  (text "Jan 10th 2024" (at 207.01 194.31 0)
-    (effects (font (size 1.27 1.27)) (justify left bottom))
-  )
-  (text "Riya Gupta LED Light Schematic" (at 187.96 190.5 0)
-    (effects (font (size 1.27 1.27)) (justify left bottom))
   )
   (hierarchical_label "VDD" (shape output) (at 157.48 71.12 0)
@@
   (symbol (lib_id "power:+5V") (at 120.65 67.31 0) (unit 1)
     (in_bom yes) (on_board yes) (fields_autoplaced)
-    (property "Reference" "#PWR?" (id 0) (at 120.65 71.12 0)
+    (property "Reference" "#PWR0121" (id 0) (at 120.65 71.12 0)
       (effects (font (size 1.27 1.27)) hide)
     )
@@
   (symbol (lib_id "power:GND") (at 123.19 82.55 0) (unit 1)
     (in_bom yes) (on_board yes) (fields_autoplaced)
-    (property "Reference" "#PWR?" (id 0) (at 123.19 88.9 0)
+    (property "Reference" "#PWR0120" (id 0) (at 123.19 88.9 0)
       (effects (font (size 1.27 1.27)) hide)
     )
@@
     (pin "1")
   )
+  (symbol (lib_id "power:+3.3V") (at 154.94 68.58 0) (unit 1)
+    (in_bom yes) (on_board yes) (fields_autoplaced)
+    (property "Reference" "#PWR0118" (id 0) (at 154.94 72.39 0)
+      (effects (font (size 1.27 1.27)) hide)
+    )
+    (property "Value" "+3.3V" (id 1) (at 154.94 63.5 0))
+    (property "Footprint" "" (id 2) (at 154.94 68.58 0)
+      (effects (font (size 1.27 1.27)) hide)
+    )
+    (property "Datasheet" "" (id 3) (at 154.94 68.58 0)
+      (effects (font (size 1.27 1.27)) hide)
+    )
+    (pin "1")
+  )
   (symbol (lib_id "power:GND") (at 151.13 83.82 0) (unit 1)
     (in_bom yes) (on_board yes) (fields_autoplaced)
-    (property "Reference" "#PWR?" (id 0) (at 151.13 90.17 0)
+    (property "Reference" "#PWR0119" (id 0) (at 151.13 90.17 0)
       (effects (font (size 1.27 1.27)) hide)
     )

Commit message: Footprints
Parts:
- C3: renamed from C11; footprint (none) -> Capacitor_SMD:C_0603_1608Metric
- C4: renamed from C10; footprint (none) -> Capacitor_SMD:C_0603_1608Metric
Changed lines of the file:
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@@
   (symbol (lib_id "Device:C_Small") (at 123.19 80.01 0) (unit 1)
     (in_bom yes) (on_board yes)
-    (property "Reference" "C11" (id 0) (at 125.73 78.7462 0)
+    (property "Reference" "C3" (id 0) (at 125.73 78.7462 0)
       (effects (font (size 1.27 1.27)) (justify left))
     )
@@
       (effects (font (size 1.27 1.27)) (justify left))
     )
-    (property "Footprint" "" (id 2) (at 123.19 80.01 0)
+    (property "Footprint" "Capacitor_SMD:C_0603_1608Metric" (id 2) (at 123.19 80.01 0)
       (effects (font (size 1.27 1.27)) hide)
     )
@@
   (symbol (lib_id "Device:C_Small") (at 151.13 76.2 0) (unit 1)
     (in_bom yes) (on_board yes)
-    (property "Reference" "C10" (id 0) (at 153.67 74.9362 0)
+    (property "Reference" "C4" (id 0) (at 153.67 74.9362 0)
       (effects (font (size 1.27 1.27)) (justify left))
     )
@@
       (effects (font (size 1.27 1.27)) (justify left))
     )
-    (property "Footprint" "" (id 2) (at 151.13 76.2 0)
+    (property "Footprint" "Capacitor_SMD:C_0603_1608Metric" (id 2) (at 151.13 76.2 0)
       (effects (font (size 1.27 1.27)) hide)
     )

Commit message: Layout
Parts:
- U2: footprint AP2112K-3.3TRG1:SOT95P285X140-5N -> AP2112K_3_3TRG1 (3):SOT95P285X140-5N
Changed lines of the file:
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@@
     (property "Reference" "U2" (id 0) (at 138.43 63.5 0))
     (property "Value" "AP2112K-3.3TRG1" (id 1) (at 138.43 66.04 0))
-    (property "Footprint" "AP2112K-3.3TRG1:SOT95P285X140-5N" (id 2) (at 138.43 76.2 0)
+    (property "Footprint" "AP2112K_3_3TRG1 (3):SOT95P285X140-5N" (id 2) (at 138.43 76.2 0)
       (effects (font (size 1.27 1.27)) (justify bottom) hide)
     )
