File: PCB Class/PCB Class.kicad_pcb (KiCad board)
At the start: 2 copper layers, 2 parts

Commit message: Layout
Parts:
- added C1: 1uF, Capacitor_SMD:C_0603_1608Metric, F.Cu at (134.6, 40.0)
- added C10: 10uF, Capacitor_SMD:C_0603_1608Metric, F.Cu at (166.6, 85.6)
- added C11: 0.1uF, Capacitor_SMD:C_0603_1608Metric, F.Cu at (187.5, 85.9)
- added C12: 10uF, Capacitor_SMD:C_0603_1608Metric, F.Cu at (191.8, 85.9)
- added C13: 0.1uF, Capacitor_SMD:C_0603_1608Metric, F.Cu at (113.3, 112.5)
- added C14: 10uF, Capacitor_SMD:C_0603_1608Metric, F.Cu at (117.1, 112.5)
- added C15: 0.1uF, Capacitor_SMD:C_0603_1608Metric, F.Cu at (138.2, 112.3)
- added C16: 10uF, Capacitor_SMD:C_0603_1608Metric, F.Cu at (142.1, 112.3)
- added C17: 0.1uF, Capacitor_SMD:C_0603_1608Metric, F.Cu at (163.1, 112.3)
- added C18: 10uF, Capacitor_SMD:C_0603_1608Metric, F.Cu at (167.4, 112.3)
- added C19: 0.1uF, Capacitor_SMD:C_0603_1608Metric, F.Cu at (186.9, 112.0)
- added C20: 10uF, Capacitor_SMD:C_0603_1608Metric, F.Cu at (191.1, 112.0)
- added C3: 22uF, Capacitor_SMD:C_0603_1608Metric, F.Cu at (111.8, 55.9)
- added C4: 22uF, Capacitor_SMD:C_0603_1608Metric, F.Cu at (111.5, 45.5)
- added C5: 0.1uF, Capacitor_SMD:C_0603_1608Metric, F.Cu at (112.3, 85.9)
- added C6: 10uF, Capacitor_SMD:C_0603_1608Metric, F.Cu at (115.3, 85.9)
- added C7: 0.1uF, Capacitor_SMD:C_0603_1608Metric, F.Cu at (137.2, 85.6)
- added C8: 10uF, Capacitor_SMD:C_0603_1608Metric, F.Cu at (140.7, 85.6)
- added J1: USB_C_Receptacle_USB2.0, Connector_USB:USB_C_Receptacle_GCT_USB4085, F.Cu at (185.1, 44.4)
- added R1: 5.1K, Resistor_SMD:R_0603_1608Metric, F.Cu at (175.0, 41.4)
- added R10: 12k, Resistor_SMD:R_0603_1608Metric, F.Cu at (182.9, 112.0)
- added R11: 10K, Resistor_SMD:R_0603_1608Metric, F.Cu at (134.6, 44.2)
- added R2: 5.1K, Resistor_SMD:R_0603_1608Metric, F.Cu at (183.4, 48.3)
- added R3: 12k, Resistor_SMD:R_0603_1608Metric, F.Cu at (109.0, 85.9)
- added R4: 12k, Resistor_SMD:R_0603_1608Metric, F.Cu at (133.7, 85.6)
- added R5: 12k, Resistor_SMD:R_0603_1608Metric, F.Cu at (158.5, 85.6)
- added R6: 12k, Resistor_SMD:R_0603_1608Metric, F.Cu at (183.1, 85.9)
- added R8: 12k, Resistor_SMD:R_0603_1608Metric, F.Cu at (134.4, 112.3)
- added R9: 12k, Resistor_SMD:R_0603_1608Metric, F.Cu at (159.0, 112.3)
- added SW1: SW_Push, Button_Switch_SMD:SW_SPST_FSMSM, F.Cu at (124.5, 44.7)
- added U1: ESP32-S3-WROOM-1-N4, ESP32_S3_WROOM_1_N4 (1):XCVR_ESP32-S3-WROOM-1-N4, F.Cu at (150.4, 45.0)
- added U10: MAX7219, MAX7219:SOIC24, F.Cu at (186.2, 102.6)
- added U2: AP2112K-3.3TRG1, AP2112K_3_3TRG1 (3):SOT95P285X140-5N, F.Cu at (112.0, 50.8)
- added U3: MAX7219, MAX7219:SOIC24, F.Cu at (111.8, 77.0)
- added U4: MAX7219, MAX7219:SOIC24, F.Cu at (136.4, 76.5)
- added U5: MAX7219, MAX7219:SOIC24, F.Cu at (162.3, 76.5)
- added U6: MAX7219, MAX7219:SOIC24, F.Cu at (186.7, 76.5)
- added U7: MAX7219, MAX7219:SOIC24, F.Cu at (111.5, 103.4)
- added U8: MAX7219, MAX7219:SOIC24, F.Cu at (136.9, 103.1)
- added U9: MAX7219, MAX7219:SOIC24, F.Cu at (162.1, 102.9)
- C9: value 100nF -> 0.1uF; footprint Capacitor_SMD:C_0402_1005Metric -> Capacitor_SMD:C_0603_1608Metric
- R7: value 10K -> 12k; footprint Resistor_SMD:R_0402_1005Metric -> Resistor_SMD:R_0603_1608Metric
- moved C9 49.6 mm to (162.8, 85.6), turned to -90 degrees
- moved R7 9.83 mm to (109.5, 112.5), turned to 90 degrees
Connections:
- C9 pad 1: /ESP32/RST -> +5V
- R7 pad 1: +3.3V -> +5V
- R7 pad 2: /ESP32/RST -> Net-(R7-Pad2)
Routing:
- net /ESP32/CLK: track 0.00 -> 218.2 mm
- net GND: track 0.00 -> 111.5 mm, vias 0 -> 36
- net /ESP32/LOAD5: track 0.00 -> 73.5 mm, vias 0 -> 2
- net /ESP32/DIN5: track 0.00 -> 61.5 mm, vias 0 -> 2
- net +5V: track 0.00 -> 61.0 mm, vias 0 -> 1
- net /ESP32/DIN8: track 0.00 -> 58.5 mm, vias 0 -> 2
- net /ESP32/LOAD8: track 0.00 -> 53.3 mm, vias 0 -> 2
- net /ESP32/D+: track 0.00 -> 52.8 mm, vias 0 -> 1
- net /ESP32/LOAD1: track 0.00 -> 52.1 mm
- net /ESP32/D-: track 0.00 -> 51.4 mm, vias 0 -> 1
- net /ESP32/LOAD6: track 0.00 -> 51.1 mm, vias 0 -> 2
- net /ESP32/DIN7: track 0.00 -> 48.9 mm, vias 0 -> 2
- net /ESP32/LOAD7: track 0.00 -> 43.6 mm, vias 0 -> 2
- net /ESP32/DIN4: track 0.00 -> 42.3 mm
- net /ESP32/DIN6: track 0.00 -> 41.5 mm, vias 0 -> 2
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- added copper zone on F.Cu, net +3.3V
- added copper zone on F.Cu, net +5V
- added copper zone on B.Cu, net GND
Other:
- board outline added: 100 x 85.8 mm
- board text added: "3.3V Regulator Room"
- board text added: "ESP Room"
- board text added: "LED Drivers Room"
- board text added: "USB Room"

Commit message: Layout V2
Parts:
- moved SW1 4.32 mm to (124.5, 49.0)
- turned C4 to -90 degrees
Routing:
- net +5V: track 61.0 -> 370.7 mm, vias 1 -> 8
- net +3.3V: track 6.69 -> 41.9 mm
- net GND: track 111.5 -> 106.6 mm, vias 36 -> 99
- net /ESP32/RST: track 17.2 -> 19.0 mm
- net /ESP32/D-: track 51.4 -> 51.9 mm
- added copper zone on F.Cu, net GND
- removed copper zone on F.Cu, net +3.3V
- removed copper zone on F.Cu, net +5V

Commit message: Final Layout
Parts:
- added BOOT: SW_Push, Button_Switch_SMD:SW_SPST_FSMSM, F.Cu at (166.9, 59.7)
- added J10: Conn_01x08_Female, Connector_PinHeader_2.54mm:PinHeader_1x08_P2.54mm_Vertical, F.Cu at (121.7, 96.5)
- added J11: Conn_01x08_Female, Connector_PinHeader_2.54mm:PinHeader_1x08_P2.54mm_Vertical, F.Cu at (103.6, 120.1)
- added J12: Conn_01x08_Female, Connector_PinHeader_2.54mm:PinHeader_1x08_P2.54mm_Vertical, F.Cu at (170.7, 96.5)
- added J13: Conn_01x08_Female, Connector_PinHeader_2.54mm:PinHeader_1x08_P2.54mm_Vertical, F.Cu at (152.9, 120.1)
- added J14: Conn_01x08_Female, Connector_PinHeader_2.54mm:PinHeader_1x08_P2.54mm_Vertical, F.Cu at (146.0, 96.5)
- added J15: Conn_01x08_Female, Connector_PinHeader_2.54mm:PinHeader_1x08_P2.54mm_Vertical, F.Cu at (128.0, 120.1)
- added J16: Conn_01x08_Female, Connector_PinHeader_2.54mm:PinHeader_1x08_P2.54mm_Vertical, F.Cu at (194.5, 96.5)
- added J17: Conn_01x08_Female, Connector_PinHeader_2.54mm:PinHeader_1x08_P2.54mm_Vertical, F.Cu at (176.5, 120.1)
- added J2: Conn_01x08_Female, Connector_PinHeader_2.54mm:PinHeader_1x08_P2.54mm_Vertical, F.Cu at (121.9, 67.1)
- added J3: Conn_01x08_Female, Connector_PinHeader_2.54mm:PinHeader_1x08_P2.54mm_Vertical, F.Cu at (103.9, 91.4)
- added J4: Conn_01x08_Female, Connector_PinHeader_2.54mm:PinHeader_1x08_P2.54mm_Vertical, F.Cu at (146.6, 67.1)
- added J5: Conn_01x08_Female, Connector_PinHeader_2.54mm:PinHeader_1x08_P2.54mm_Vertical, F.Cu at (128.3, 91.4)
- added J6: Conn_01x08_Female, Connector_PinHeader_2.54mm:PinHeader_1x08_P2.54mm_Vertical, F.Cu at (171.2, 67.1)
- added J7: Conn_01x08_Female, Connector_PinHeader_2.54mm:PinHeader_1x08_P2.54mm_Vertical, F.Cu at (152.9, 91.2)
- added J8: Conn_01x08_Female, Connector_PinHeader_2.54mm:PinHeader_1x08_P2.54mm_Vertical, F.Cu at (195.8, 67.1)
- added J9: Conn_01x08_Female, Connector_PinHeader_2.54mm:PinHeader_1x08_P2.54mm_Vertical, F.Cu at (176.8, 90.9)
- added REF**: EdgertonLogo, Logos:EdgertonLogo2, F.Cu at (100.7, 54.4)
- added REF**: MechELogo, Logos:MechELogo, F.Cu at (101.2, 46.3)
- moved R3 12.8 mm to (120.7, 80.5), turned to 180 degrees
- moved R6 12.6 mm to (194.6, 80.6), turned to 180 degrees
- moved R5 12.3 mm to (169.9, 80.8), turned to 180 degrees
- moved C5 12.1 mm to (121.9, 78.5), turned to 0 degrees
- moved R4 12.1 mm to (144.8, 80.8), turned to 180 degrees
- moved C7 11.6 mm to (146.6, 78.7), turned to 0 degrees
- moved R7 11.2 mm to (120.4, 110.4), turned to 180 degrees
- moved R10 11.1 mm to (193.8, 110.2), turned to 180 degrees
- moved C9 11.0 mm to (171.4, 78.7), turned to 0 degrees
- moved C11 10.9 mm to (195.9, 78.9), turned to 0 degrees
- moved R8 10.9 mm to (145.0, 110.1), turned to 180 degrees
- moved C6 10.6 mm to (120.7, 76.7), turned to 0 degrees
- moved R9 10.5 mm to (169.2, 110.0), turned to 180 degrees
- moved C12 9.94 mm to (194.6, 76.3), turned to 0 degrees
- moved C8 9.77 mm to (144.8, 76.7), turned to 0 degrees
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- renumbered SW1 to RST
Connections:
- U1 pad 16: /ESP32/LOAD6 -> /ESP32/LOAD2
- U1 pad 17: /ESP32/DIN6 -> /ESP32/DIN2
- U1 pad 18: /ESP32/LOAD7 -> /ESP32/CLK
- U1 pad 19: /ESP32/DIN7 -> /ESP32/LOAD7
- U1 pad 20: /ESP32/CLK -> /ESP32/DIN7
- U1 pad 27: unconnected-(U1-Pad27) -> Net-(SW2-Pad2)
- U1 pad 4: /ESP32/LOAD1 -> /ESP32/LOAD5
- U1 pad 5: /ESP32/DIN1 -> /ESP32/DIN5
- U1 pad 6: /ESP32/LOAD5 -> /ESP32/LOAD1
- U1 pad 7: /ESP32/DIN5 -> /ESP32/DIN1
- U1 pad 8: /ESP32/LOAD2 -> /ESP32/LOAD6
- U1 pad 9: /ESP32/DIN2 -> /ESP32/DIN6
- U10 pad 10: /LED Driver2/R86 -> /LED Driver2/R87
- U10 pad 11: /LED Driver2/R82 -> /LED Driver2/R88
- U10 pad 15: /LED Driver2/C86 -> /LED Driver2/C82
- U10 pad 16: /LED Driver2/C82 -> /LED Driver2/C83
- U10 pad 17: /LED Driver2/C87 -> /LED Driver2/C84
- U10 pad 20: /LED Driver2/C83 -> /LED Driver2/C85
- U10 pad 21: /LED Driver2/C85 -> /LED Driver2/C86
- U10 pad 22: /LED Driver2/C88 -> /LED Driver2/C87
- U10 pad 23: /LED Driver2/C84 -> /LED Driver2/C88
- U10 pad 3: /LED Driver2/R85 -> /LED Driver2/R82
- U10 pad 5: /LED Driver2/R87 -> /LED Driver2/R83
- U10 pad 6: /LED Driver2/R83 -> /LED Driver2/R84
- U10 pad 7: /LED Driver2/R84 -> /LED Driver2/R85
- U10 pad 8: /LED Driver2/R88 -> /LED Driver2/R86
- U3 pad 10: /LED Driver/R16 -> /LED Driver/R17
- U3 pad 11: /LED Driver/R12 -> /LED Driver/R18
- U3 pad 15: /LED Driver/C16 -> /LED Driver/C12
- U3 pad 16: /LED Driver/C12 -> /LED Driver/C13
- U3 pad 17: /LED Driver/C17 -> /LED Driver/C14
- U3 pad 20: /LED Driver/C13 -> /LED Driver/C15
- U3 pad 21: /LED Driver/C15 -> /LED Driver/C16
- U3 pad 22: /LED Driver/C18 -> /LED Driver/C17
- U3 pad 23: /LED Driver/C14 -> /LED Driver/C18
- U3 pad 3: /LED Driver/R15 -> /LED Driver/R12
- U3 pad 5: /LED Driver/R17 -> /LED Driver/R13
- U3 pad 6: /LED Driver/R13 -> /LED Driver/R14
- U3 pad 7: /LED Driver/R14 -> /LED Driver/R15
- U3 pad 8: /LED Driver/R18 -> /LED Driver/R16
- U4 pad 10: /LED Driver/R26 -> /LED Driver/R27
- U4 pad 11: /LED Driver/R22 -> /LED Driver/R28
- U4 pad 15: /LED Driver/C26 -> /LED Driver/C22
- U4 pad 16: /LED Driver/C22 -> /LED Driver/C23
- U4 pad 17: /LED Driver/C27 -> /LED Driver/C24
- U4 pad 20: /LED Driver/C23 -> /LED Driver/C25
- U4 pad 21: /LED Driver/C25 -> /LED Driver/C26
- U4 pad 22: /LED Driver/C28 -> /LED Driver/C27
- U4 pad 23: /LED Driver/C24 -> /LED Driver/C28
- U4 pad 3: /LED Driver/R25 -> /LED Driver/R22
- U4 pad 5: /LED Driver/R27 -> /LED Driver/R23
- U4 pad 6: /LED Driver/R23 -> /LED Driver/R24
- U4 pad 7: /LED Driver/R24 -> /LED Driver/R25
- U4 pad 8: /LED Driver/R28 -> /LED Driver/R26
- U5 pad 10: /LED Driver/R36 -> /LED Driver/R37
- U5 pad 11: /LED Driver/R32 -> /LED Driver/R38
- U5 pad 15: /LED Driver/C36 -> /LED Driver/C32
- U5 pad 16: /LED Driver/C32 -> /LED Driver/C33
- U5 pad 17: /LED Driver/C37 -> /LED Driver/C34
- U5 pad 20: /LED Driver/C33 -> /LED Driver/C35
- U5 pad 21: /LED Driver/C35 -> /LED Driver/C36
- U5 pad 22: /LED Driver/C38 -> /LED Driver/C37
- U5 pad 23: /LED Driver/C34 -> /LED Driver/C38
- U5 pad 3: /LED Driver/R35 -> /LED Driver/R32
- U5 pad 5: /LED Driver/R37 -> /LED Driver/R33
- U5 pad 6: /LED Driver/R33 -> /LED Driver/R34
- U5 pad 7: /LED Driver/R34 -> /LED Driver/R35
- U5 pad 8: /LED Driver/R38 -> /LED Driver/R36
- U6 pad 10: /LED Driver/R46 -> /LED Driver/R47
- U6 pad 11: /LED Driver/R42 -> /LED Driver/R48
- U6 pad 15: /LED Driver/C46 -> /LED Driver/C42
- U6 pad 16: /LED Driver/C42 -> /LED Driver/C43
- U6 pad 17: /LED Driver/C47 -> /LED Driver/C44
- U6 pad 20: /LED Driver/C43 -> /LED Driver/C45
- U6 pad 21: /LED Driver/C45 -> /LED Driver/C46
- U6 pad 22: /LED Driver/C48 -> /LED Driver/C47
- U6 pad 23: /LED Driver/C44 -> /LED Driver/C48
- U6 pad 3: /LED Driver/R45 -> /LED Driver/R42
- U6 pad 5: /LED Driver/R47 -> /LED Driver/R43
- U6 pad 6: /LED Driver/R43 -> /LED Driver/R44
- U6 pad 7: /LED Driver/R44 -> /LED Driver/R45
- U6 pad 8: /LED Driver/R48 -> /LED Driver/R46
- U7 pad 10: /LED Driver2/R56 -> /LED Driver2/R57
- U7 pad 11: /LED Driver2/R52 -> /LED Driver2/R58
- U7 pad 15: /LED Driver2/C56 -> /LED Driver2/C52
- U7 pad 16: /LED Driver2/C52 -> /LED Driver2/C53
- U7 pad 17: /LED Driver2/C57 -> /LED Driver2/C54
- U7 pad 20: /LED Driver2/C53 -> /LED Driver2/C55
- U7 pad 21: /LED Driver2/C55 -> /LED Driver2/C56
- U7 pad 22: /LED Driver2/C58 -> /LED Driver2/C57
- U7 pad 23: /LED Driver2/C54 -> /LED Driver2/C58
- U7 pad 3: /LED Driver2/R55 -> /LED Driver2/R52
- U7 pad 5: /LED Driver2/R57 -> /LED Driver2/R53
- U7 pad 6: /LED Driver2/R53 -> /LED Driver2/R54
- U7 pad 7: /LED Driver2/R54 -> /LED Driver2/R55
- U7 pad 8: /LED Driver2/R58 -> /LED Driver2/R56
- U8 pad 10: /LED Driver2/R66 -> /LED Driver2/R67
- U8 pad 11: /LED Driver2/R62 -> /LED Driver2/R68
- U8 pad 15: /LED Driver2/C66 -> /LED Driver2/C62
- U8 pad 16: /LED Driver2/C62 -> /LED Driver2/C63
- U8 pad 17: /LED Driver2/C67 -> /LED Driver2/C64
- U8 pad 20: /LED Driver2/C63 -> /LED Driver2/C65
- U8 pad 21: /LED Driver2/C65 -> /LED Driver2/C66
- U8 pad 22: /LED Driver2/C68 -> /LED Driver2/C67
- U8 pad 23: /LED Driver2/C64 -> /LED Driver2/C68
- U8 pad 3: /LED Driver2/R65 -> /LED Driver2/R62
- U8 pad 5: /LED Driver2/R67 -> /LED Driver2/R63
- U8 pad 6: /LED Driver2/R63 -> /LED Driver2/R64
- U8 pad 7: /LED Driver2/R64 -> /LED Driver2/R65
- U8 pad 8: /LED Driver2/R68 -> /LED Driver2/R66
- U9 pad 10: /LED Driver2/R76 -> /LED Driver2/R77
- U9 pad 11: /LED Driver2/R72 -> /LED Driver2/R78
- U9 pad 15: /LED Driver2/C76 -> /LED Driver2/C72
- U9 pad 16: /LED Driver2/C72 -> /LED Driver2/C73
- U9 pad 17: /LED Driver2/C77 -> /LED Driver2/C74
- U9 pad 20: /LED Driver2/C73 -> /LED Driver2/C75
- U9 pad 21: /LED Driver2/C75 -> /LED Driver2/C76
- U9 pad 22: /LED Driver2/C78 -> /LED Driver2/C77
- U9 pad 23: /LED Driver2/C74 -> /LED Driver2/C78
- U9 pad 3: /LED Driver2/R75 -> /LED Driver2/R72
- U9 pad 5: /LED Driver2/R77 -> /LED Driver2/R73
- U9 pad 6: /LED Driver2/R73 -> /LED Driver2/R74
- U9 pad 7: /LED Driver2/R74 -> /LED Driver2/R75
- U9 pad 8: /LED Driver2/R78 -> /LED Driver2/R76
Routing:
- net /ESP32/CLK: track 218.2 -> 312.1 mm, vias 0 -> 6
- net GND: track 106.6 -> 30.5 mm, vias 99 -> 107
- net +5V: track 370.7 -> 423.4 mm, vias 8 -> 15
- net /ESP32/LOAD5: track 73.5 -> 105.7 mm, vias 2 -> 0
- net /ESP32/DIN5: track 61.5 -> 90.5 mm, vias 2 -> 0
- net /ESP32/LOAD6: track 51.1 -> 79.5 mm, vias 2 -> 0
- net /ESP32/LOAD8: track 53.3 -> 78.8 mm, vias 2 -> 0
- net /ESP32/LOAD4: track 27.4 -> 51.1 mm
- net /ESP32/DIN6: track 41.5 -> 64.2 mm, vias 2 -> 0
- net /ESP32/LOAD1: track 52.1 -> 73.5 mm
- net /ESP32/LOAD2: track 28.5 -> 48.5 mm
- net /ESP32/DIN1: track 37.9 -> 57.4 mm
- net /ESP32/LOAD7: track 43.6 -> 61.5 mm, vias 2 -> 0
- net /ESP32/LOAD3: track 15.7 -> 32.6 mm
- net /LED Driver2/R54: track 0.00 -> 15.3 mm
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Other:
- board text added: "Riya Gupta LED Cube Controller MIT PCB Class 2024"
