File: PCB Class/driver1.kicad_sch (KiCad schematic)
At the start: 4 parts, among them U3 MAX7219

Commit message: Final Schematic
Parts:
- added C1, C5, C7: 0.1uF, symbol Device:C_Small
- added C4, C6, C8: 10uF, symbol Device:C_Polarized_Small_US
- added R4, R5, R6: 33k, symbol Device:R_Small
- added U4, U5, U6: MAX7219, symbol Driver_LED:MAX7219
Connections:
- net +5V: now also C1.1, C4.1, C5.1, C6.1, C7.1, C8.1, R4.1, R5.1, R6.1, U4.19 (V+), U5.19 (V+), U6.19 (V+)
- net GND: now also C1.2, C4.2, C5.2, C6.2, C7.2, C8.2, U4.4 (GND), U4.9 (GND), U5.4 (GND), U5.9 (GND), U6.4 (GND), U6.9 (GND)
- net C1 1-8 renamed C11
- net C2 1-8 renamed C12
- net C3 1-8 renamed C13
- net C4 1-8 renamed C14
- net C5 1-8 renamed C15
- net C6 1-8 renamed C16
- net C7 1-8 renamed C17
- net C8 1-8 renamed C18
- net CLK1 renamed CLK
- net CLK: now also U4.13 (CLK), U5.13 (CLK), U6.13 (CLK)
- net R1 1-8 renamed R11
- net R2 1-8 renamed R12
- net R3 1-8 renamed R13
- net R4 1-8 renamed R14
- net R5 1-8 renamed R15
- net R6 1-8 renamed R16
- net R7 1-8 renamed R17
- net R8 1-8 renamed R18
- new net: R6.2, U6.18 (ISET)
- new net: R4.2, U4.18 (ISET)
- new net: R5.2, U5.18 (ISET)
- new net C21: U5.14 (SEG_A)
- new net C22: U5.16 (SEG_B)
- new net C23: U5.20 (SEG_C)
- new net C24: U5.23 (SEG_D)
- new net C25: U5.21 (SEG_E)
- new net C26: U5.15 (SEG_F)
- new net C27: U5.17 (SEG_G)
- new net C28: U5.22 (SEG_DP)
- new net C31: U6.14 (SEG_A)
- new net C32: U6.16 (SEG_B)
- new net C33: U6.20 (SEG_C)
- new net C34: U6.23 (SEG_D)
- new net C35: U6.21 (SEG_E)
- new net C36: U6.15 (SEG_F)
- new net C37: U6.17 (SEG_G)
- new net C38: U6.22 (SEG_DP)
- new net C41: U4.14 (SEG_A)
- new net C42: U4.16 (SEG_B)
- new net C43: U4.20 (SEG_C)
- new net C44: U4.23 (SEG_D)
- new net C45: U4.21 (SEG_E)
- new net C46: U4.15 (SEG_F)
- new net C47: U4.17 (SEG_G)
- new net C48: U4.22 (SEG_DP)
- new net DIN2: U5.1 (DIN)
- new net DIN3: U6.1 (DIN)
- new net DIN4: U4.1 (DIN)
- new net LOAD2: U5.12 (LOAD)
- new net LOAD3: U6.12 (LOAD)
- new net LOAD4: U4.12 (LOAD)
- new net R21: U5.2 (DIG_0)
- new net R22: U5.11 (DIG_1)
- new net R23: U5.6 (DIG_2)
- new net R24: U5.7 (DIG_3)
- new net R25: U5.3 (DIG_4)
- new net R26: U5.10 (DIG_5)
- new net R27: U5.5 (DIG_6)
- new net R28: U5.8 (DIG_7)
- new net R31: U6.2 (DIG_0)
- new net R32: U6.11 (DIG_1)
- new net R33: U6.6 (DIG_2)
- new net R34: U6.7 (DIG_3)
- new net R35: U6.3 (DIG_4)
- new net R36: U6.10 (DIG_5)
- new net R37: U6.5 (DIG_6)
- new net R38: U6.8 (DIG_7)
- new net R41: U4.2 (DIG_0)
- new net R42: U4.11 (DIG_1)
- new net R43: U4.6 (DIG_2)
- new net R44: U4.7 (DIG_3)
- new net R45: U4.3 (DIG_4)
- new net R46: U4.10 (DIG_5)
- new net R47: U4.5 (DIG_6)
- new net R48: U4.8 (DIG_7)
- no-connect marks 1 -> 4
Other:
- note removed: "Jan 10th 2024"
- note removed: "Riya Gupta LED Light Schematic"
- title: (none) -> RGB LED Lights
- moved on the sheet: C2, C3, R3, U3

Commit message: Footprints
Parts:
- C10: renamed from C8; footprint (none) -> Capacitor_SMD:C_0603_1608Metric
- C11: renamed from C1; footprint (none) -> Capacitor_SMD:C_0603_1608Metric
- C12: renamed from C4; footprint (none) -> Capacitor_SMD:C_0603_1608Metric
- C5: renamed from C2; footprint (none) -> Capacitor_SMD:C_0603_1608Metric
- C6: renamed from C3; footprint (none) -> Capacitor_SMD:C_0603_1608Metric
- C7: renamed from C5; footprint (none) -> Capacitor_SMD:C_0603_1608Metric
- C8: renamed from C6; footprint (none) -> Capacitor_SMD:C_0603_1608Metric
- C9: renamed from C7; footprint (none) -> Capacitor_SMD:C_0603_1608Metric
- R4: renamed from R3; value 33k -> 12k; footprint (none) -> Resistor_SMD:R_0603_1608Metric
- R5, R6: value 33k -> 12k; footprint (none) -> Resistor_SMD:R_0603_1608Metric
- R7: renamed from R4; value 33k -> 12k; footprint (none) -> Resistor_SMD:R_0603_1608Metric
- U3, U4, U5, U6: footprint (none) -> MAX7219:SOIC24
Other:
- moved on the sheet: C10, C11, C12, C7, C8, C9, R5, R6, R7, U4, U5, U6

Commit message: Layout
Parts:
- renumbered R4 to R3, R5 to R4, R6 to R5, R7 to R6, U5 to U4, U6 to U5, U4 to U6
Changed lines of the file:
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@@
   (symbol (lib_id "Device:R_Small") (at 48.26 109.22 0) (unit 1)
     (in_bom yes) (on_board yes) (fields_autoplaced)
-    (property "Reference" "R6" (id 0) (at 50.8 107.9499 0)
+    (property "Reference" "R5" (id 0) (at 50.8 107.9499 0)
       (effects (font (size 1.27 1.27)) (justify left))
     )
@@
   (symbol (lib_id "Driver_LED:MAX7219") (at 139.7 130.81 0) (unit 1)
     (in_bom yes) (on_board yes) (fields_autoplaced)
-    (property "Reference" "U4" (id 0) (at 141.7194 102.87 0)
+    (property "Reference" "U6" (id 0) (at 141.7194 102.87 0)
       (effects (font (size 1.27 1.27)) (justify left))
     )
@@
   (symbol (lib_id "Device:R_Small") (at 119.38 30.48 0) (unit 1)
     (in_bom yes) (on_board yes) (fields_autoplaced)
-    (property "Reference" "R5" (id 0) (at 121.92 29.2099 0)
+    (property "Reference" "R4" (id 0) (at 121.92 29.2099 0)
       (effects (font (size 1.27 1.27)) (justify left))
     )
@@
   (symbol (lib_id "Device:R_Small") (at 46.99 30.48 0) (unit 1)
     (in_bom yes) (on_board yes) (fields_autoplaced)
-    (property "Reference" "R4" (id 0) (at 49.53 29.2099 0)
+    (property "Reference" "R3" (id 0) (at 49.53 29.2099 0)
       (effects (font (size 1.27 1.27)) (justify left))
     )
@@
   (symbol (lib_id "Driver_LED:MAX7219") (at 64.77 133.35 0) (unit 1)
     (in_bom yes) (on_board yes) (fields_autoplaced)
-    (property "Reference" "U6" (id 0) (at 66.7894 105.41 0)
+    (property "Reference" "U5" (id 0) (at 66.7894 105.41 0)
       (effects (font (size 1.27 1.27)) (justify left))
     )
@@
   (symbol (lib_id "Driver_LED:MAX7219") (at 135.89 54.61 0) (unit 1)
     (in_bom yes) (on_board yes) (fields_autoplaced)
-    (property "Reference" "U5" (id 0) (at 137.9094 26.67 0)
+    (property "Reference" "U4" (id 0) (at 137.9094 26.67 0)
       (effects (font (size 1.27 1.27)) (justify left))
     )
@@
   (symbol (lib_id "Device:R_Small") (at 123.19 106.68 0) (unit 1)
     (in_bom yes) (on_board yes) (fields_autoplaced)
-    (property "Reference" "R7" (id 0) (at 125.73 105.4099 0)
-      (effects (font (size 1.27 1.27)) (justify left))
-    )
+    (property "Reference" "R6" (id 0) (at 125.73 105.4099 0)
+      (effects (font (size 1.27 1.27)) (justify left))
+    )

Commit message: Final Layout
Parts:
- added J2, J3, J4, J5, J6, J7, J8, J9: Conn_01x08_Female, Connector_PinHeader_2.54mm:PinHeader_1x08_P2.54mm_Vertical, symbol Connector:Conn_01x08_Female
Connections:
- net C11: now also J3.8 (Pin_8)
- net C12: now also U3.15 (SEG_F), J3.7 (Pin_7); no longer U3.16 (SEG_B)
- net C13: now also U3.16 (SEG_B), J3.6 (Pin_6); no longer U3.20 (SEG_C)
- net C14: now also U3.17 (SEG_G), J3.5 (Pin_5); no longer U3.23 (SEG_D)
- net C15: now also U3.20 (SEG_C), J2.4 (Pin_4); no longer U3.21 (SEG_E)
- net C16: now also U3.21 (SEG_E), J2.3 (Pin_3); no longer U3.15 (SEG_F)
- net C17: now also U3.22 (SEG_DP), J2.2 (Pin_2); no longer U3.17 (SEG_G)
- net C18: now also U3.23 (SEG_D), J2.1 (Pin_1); no longer U3.22 (SEG_DP)
- net C21: now also J5.8 (Pin_8)
- net C22: now also U4.15 (SEG_F), J5.7 (Pin_7); no longer U4.16 (SEG_B)
- net C23: now also U4.16 (SEG_B), J5.6 (Pin_6); no longer U4.20 (SEG_C)
- net C24: now also U4.17 (SEG_G), J5.5 (Pin_5); no longer U4.23 (SEG_D)
- net C25: now also U4.20 (SEG_C), J4.4 (Pin_4); no longer U4.21 (SEG_E)
- net C26: now also U4.21 (SEG_E), J4.3 (Pin_3); no longer U4.15 (SEG_F)
- net C27: now also U4.22 (SEG_DP), J4.2 (Pin_2); no longer U4.17 (SEG_G)
- net C28: now also U4.23 (SEG_D), J4.1 (Pin_1); no longer U4.22 (SEG_DP)
- net C31: now also J7.8 (Pin_8)
- net C32: now also U5.15 (SEG_F), J7.7 (Pin_7); no longer U5.16 (SEG_B)
- net C33: now also U5.16 (SEG_B), J7.6 (Pin_6); no longer U5.20 (SEG_C)
- net C34: now also U5.17 (SEG_G), J7.5 (Pin_5); no longer U5.23 (SEG_D)
- net C35: now also U5.20 (SEG_C), J6.4 (Pin_4); no longer U5.21 (SEG_E)
- net C36: now also U5.21 (SEG_E), J6.3 (Pin_3); no longer U5.15 (SEG_F)
- net C37: now also U5.22 (SEG_DP), J6.2 (Pin_2); no longer U5.17 (SEG_G)
- net C38: now also U5.23 (SEG_D), J6.1 (Pin_1); no longer U5.22 (SEG_DP)
- net C41: now also J9.8 (Pin_8)
- net C42: now also U6.15 (SEG_F), J9.7 (Pin_7); no longer U6.16 (SEG_B)
- net C43: now also U6.16 (SEG_B), J9.6 (Pin_6); no longer U6.20 (SEG_C)
- net C44: now also U6.17 (SEG_G), J9.5 (Pin_5); no longer U6.23 (SEG_D)
- net C45: now also U6.20 (SEG_C), J8.4 (Pin_4); no longer U6.21 (SEG_E)
- net C46: now also U6.21 (SEG_E), J8.3 (Pin_3); no longer U6.15 (SEG_F)
- net C47: now also U6.22 (SEG_DP), J8.2 (Pin_2); no longer U6.17 (SEG_G)
- net C48: now also U6.23 (SEG_D), J8.1 (Pin_1); no longer U6.22 (SEG_DP)
- net R11: now also J2.8 (Pin_8)
- net R12: now also U3.3 (DIG_4), J2.7 (Pin_7); no longer U3.11 (DIG_1)
- net R13: now also U3.5 (DIG_6), J2.6 (Pin_6); no longer U3.6 (DIG_2)
- net R14: now also U3.6 (DIG_2), J2.5 (Pin_5); no longer U3.7 (DIG_3)
- net R15: now also U3.7 (DIG_3), J3.4 (Pin_4); no longer U3.3 (DIG_4)
- net R16: now also U3.8 (DIG_7), J3.3 (Pin_3); no longer U3.10 (DIG_5)
- net R17: now also U3.10 (DIG_5), J3.2 (Pin_2); no longer U3.5 (DIG_6)
- net R18: now also U3.11 (DIG_1), J3.1 (Pin_1); no longer U3.8 (DIG_7)
- net R21: now also J4.8 (Pin_8)
- net R22: now also U4.3 (DIG_4), J4.7 (Pin_7); no longer U4.11 (DIG_1)
- net R23: now also U4.5 (DIG_6), J4.6 (Pin_6); no longer U4.6 (DIG_2)
- net R24: now also U4.6 (DIG_2), J4.5 (Pin_5); no longer U4.7 (DIG_3)
- net R25: now also U4.7 (DIG_3), J5.4 (Pin_4); no longer U4.3 (DIG_4)
- net R26: now also U4.8 (DIG_7), J5.3 (Pin_3); no longer U4.10 (DIG_5)
- net R27: now also U4.10 (DIG_5), J5.2 (Pin_2); no longer U4.5 (DIG_6)
- net R28: now also U4.11 (DIG_1), J5.1 (Pin_1); no longer U4.8 (DIG_7)
- net R31: now also J6.8 (Pin_8)
- net R32: now also U5.3 (DIG_4), J6.7 (Pin_7); no longer U5.11 (DIG_1)
- net R33: now also U5.5 (DIG_6), J6.6 (Pin_6); no longer U5.6 (DIG_2)
- net R34: now also U5.6 (DIG_2), J6.5 (Pin_5); no longer U5.7 (DIG_3)
- net R35: now also U5.7 (DIG_3), J7.4 (Pin_4); no longer U5.3 (DIG_4)
- net R36: now also U5.8 (DIG_7), J7.3 (Pin_3); no longer U5.10 (DIG_5)
- net R37: now also U5.10 (DIG_5), J7.2 (Pin_2); no longer U5.5 (DIG_6)
- net R38: now also U5.11 (DIG_1), J7.1 (Pin_1); no longer U5.8 (DIG_7)
- net R41: now also J8.8 (Pin_8)
- net R42: now also U6.3 (DIG_4), J8.7 (Pin_7); no longer U6.11 (DIG_1)
- net R43: now also U6.5 (DIG_6), J8.6 (Pin_6); no longer U6.6 (DIG_2)
- net R44: now also U6.6 (DIG_2), J8.5 (Pin_5); no longer U6.7 (DIG_3)
- net R45: now also U6.7 (DIG_3), J9.4 (Pin_4); no longer U6.3 (DIG_4)
- net R46: now also U6.8 (DIG_7), J9.3 (Pin_3); no longer U6.10 (DIG_5)
- net R47: now also U6.10 (DIG_5), J9.2 (Pin_2); no longer U6.5 (DIG_6)
- net R48: now also U6.11 (DIG_1), J9.1 (Pin_1); no longer U6.8 (DIG_7)
