File: PCB Class/driver2.kicad_sch (KiCad schematic)
At the start: 4 parts, among them U4 MAX7219

Commit message: Final Schematic
Parts:
- removed C4: 0.1uF, symbol Device:C_Small
- removed C5: 10uF, symbol Device:C_Polarized_Small_US
- removed U4: MAX7219, symbol Driver_LED:MAX7219
- added C1, C2, C5, C7: 0.1uF, symbol Device:C_Small
- added C3, C4, C6, C8: 10uF, symbol Device:C_Polarized_Small_US
- added R3, R4, R6: 33k, symbol Device:R_Small
- added U10, U7, U8, U9: MAX7219, symbol Driver_LED:MAX7219
Connections:
- net +5V: now also C1.1, C2.1, C3.1, C4.1, C5.1, C6.1, C7.1, C8.1, R3.1, R4.1, R6.1, U10.19 (V+), U7.19 (V+), U8.19 (V+), U9.19 (V+)
- net GND: now also C1.2, C2.2, C3.2, C4.2, C5.2, C6.2, C7.2, C8.2, U10.4 (GND), U10.9 (GND), U7.4 (GND), U7.9 (GND), U8.4 (GND), U8.9 (GND), U9.4 (GND), U9.9 (GND)
- net at R5.2: now also U8.18 (ISET)
- new net: R6.2, U10.18 (ISET)
- new net: R4.2, U9.18 (ISET)
- new net: R3.2, U7.18 (ISET)
- new net C51: U7.14 (SEG_A)
- new net C52: U7.16 (SEG_B)
- new net C53: U7.20 (SEG_C)
- new net C54: U7.23 (SEG_D)
- new net C55: U7.21 (SEG_E)
- new net C56: U7.15 (SEG_F)
- new net C57: U7.17 (SEG_G)
- new net C58: U7.22 (SEG_DP)
- new net C61: U8.14 (SEG_A)
- new net C62: U8.16 (SEG_B)
- new net C63: U8.20 (SEG_C)
- new net C64: U8.23 (SEG_D)
- new net C65: U8.21 (SEG_E)
- new net C66: U8.15 (SEG_F)
- new net C67: U8.17 (SEG_G)
- new net C68: U8.22 (SEG_DP)
- new net C71: U9.14 (SEG_A)
- new net C72: U9.16 (SEG_B)
- new net C73: U9.20 (SEG_C)
- new net C74: U9.23 (SEG_D)
- new net C75: U9.21 (SEG_E)
- new net C76: U9.15 (SEG_F)
- new net C77: U9.17 (SEG_G)
- new net C78: U9.22 (SEG_DP)
- new net C81: U10.14 (SEG_A)
- new net C82: U10.16 (SEG_B)
- new net C83: U10.20 (SEG_C)
- new net C84: U10.23 (SEG_D)
- new net C85: U10.21 (SEG_E)
- new net C86: U10.15 (SEG_F)
- new net C87: U10.17 (SEG_G)
- new net C88: U10.22 (SEG_DP)
- new net CLK: U10.13 (CLK), U7.13 (CLK), U8.13 (CLK), U9.13 (CLK)
- new net DIN5: U7.1 (DIN)
- new net DIN6: U8.1 (DIN)
- new net DIN7: U9.1 (DIN)
- new net DIN8: U10.1 (DIN)
- new net LOAD5: U7.12 (LOAD)
- new net LOAD6: U8.12 (LOAD)
- new net LOAD7: U9.12 (LOAD)
- new net LOAD8: U10.12 (LOAD)
- new net R51: U7.2 (DIG_0)
- new net R52: U7.11 (DIG_1)
- new net R53: U7.6 (DIG_2)
- new net R54: U7.7 (DIG_3)
- new net R55: U7.3 (DIG_4)
- new net R56: U7.10 (DIG_5)
- new net R57: U7.5 (DIG_6)
- new net R58: U7.8 (DIG_7)
- new net R61: U8.2 (DIG_0)
- new net R62: U8.11 (DIG_1)
- new net R63: U8.6 (DIG_2)
- new net R64: U8.7 (DIG_3)
- new net R65: U8.3 (DIG_4)
- new net R66: U8.10 (DIG_5)
- new net R67: U8.5 (DIG_6)
- new net R68: U8.8 (DIG_7)
- new net R71: U9.2 (DIG_0)
- new net R72: U9.11 (DIG_1)
- new net R73: U9.6 (DIG_2)
- new net R74: U9.7 (DIG_3)
- new net R75: U9.3 (DIG_4)
- new net R76: U9.10 (DIG_5)
- new net R77: U9.5 (DIG_6)
- new net R78: U9.8 (DIG_7)
- new net R81: U10.2 (DIG_0)
- new net R82: U10.11 (DIG_1)
- new net R83: U10.6 (DIG_2)
- new net R84: U10.7 (DIG_3)
- new net R85: U10.3 (DIG_4)
- new net R86: U10.10 (DIG_5)
- new net R87: U10.5 (DIG_6)
- new net R88: U10.8 (DIG_7)
- no-connect marks 7 -> 4
Other:
- note removed: "Jan 10th 2024"
- note removed: "Riya Gupta LED Light Schematic"
- title: (none) -> RGB LED Lights

Commit message: Footprints
Parts:
- removed C1, C2, C5, C7: 0.1uF, symbol Device:C_Small
- removed C3, C4, C6, C8: 10uF, symbol Device:C_Polarized_Small_US
- removed R3, R4, R5, R6: 33k, symbol Device:R_Small
- added C13, C15, C17, C19: 0.1uF, Capacitor_SMD:C_0603_1608Metric, symbol Device:C_Small
- added C14, C16, C18, C20: 10uF, Capacitor_SMD:C_0603_1608Metric, symbol Device:C_Polarized_Small_US
- added R10, R11, R8, R9: 12k, Resistor_SMD:R_0603_1608Metric, symbol Device:R_Small
- U10, U7, U8, U9: footprint (none) -> MAX7219:SOIC24
Connections:
- net +5V: now also C13.1, C14.1, C15.1, C16.1, C17.1, C18.1, C19.1, C20.1, R10.1, R11.1, R8.1, R9.1
- net GND: now also C13.2, C14.2, C15.2, C16.2, C17.2, C18.2, C19.2, C20.2
- net at U10.18 (ISET): now also R11.2
- net at U9.18 (ISET): now also R10.2
- net at U8.18 (ISET): now also R9.2
- net at U7.18 (ISET): now also R8.2

Commit message: Layout
Parts:
- renumbered R11 to R10, R8 to R7, R9 to R8, R10 to R9
Changed lines of the file:
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@@
   (symbol (lib_id "Device:R_Small") (at 46.99 30.48 0) (unit 1)
     (in_bom yes) (on_board yes) (fields_autoplaced)
-    (property "Reference" "R8" (id 0) (at 49.53 29.2099 0)
+    (property "Reference" "R7" (id 0) (at 49.53 29.2099 0)
       (effects (font (size 1.27 1.27)) (justify left))
     )
@@
   (symbol (lib_id "Device:R_Small") (at 46.99 106.68 0) (unit 1)
     (in_bom yes) (on_board yes) (fields_autoplaced)
-    (property "Reference" "R10" (id 0) (at 49.53 105.4099 0)
+    (property "Reference" "R9" (id 0) (at 49.53 105.4099 0)
       (effects (font (size 1.27 1.27)) (justify left))
     )
@@
   (symbol (lib_id "Device:R_Small") (at 120.65 27.94 0) (unit 1)
     (in_bom yes) (on_board yes) (fields_autoplaced)
-    (property "Reference" "R9" (id 0) (at 123.19 26.6699 0)
+    (property "Reference" "R8" (id 0) (at 123.19 26.6699 0)
       (effects (font (size 1.27 1.27)) (justify left))
     )
@@
   (symbol (lib_id "Device:R_Small") (at 120.65 106.68 0) (unit 1)
     (in_bom yes) (on_board yes) (fields_autoplaced)
-    (property "Reference" "R11" (id 0) (at 123.19 105.4099 0)
-      (effects (font (size 1.27 1.27)) (justify left))
-    )
+    (property "Reference" "R10" (id 0) (at 123.19 105.4099 0)
+      (effects (font (size 1.27 1.27)) (justify left))
+    )

Commit message: Final Layout
Parts:
- added J10, J11, J12, J13, J14, J15, J16, J17: Conn_01x08_Female, Connector_PinHeader_2.54mm:PinHeader_1x08_P2.54mm_Vertical, symbol Connector:Conn_01x08_Female
Connections:
- net C51: now also J11.8 (Pin_8)
- net C52: now also U7.15 (SEG_F), J11.7 (Pin_7); no longer U7.16 (SEG_B)
- net C53: now also U7.16 (SEG_B), J11.6 (Pin_6); no longer U7.20 (SEG_C)
- net C54: now also U7.17 (SEG_G), J11.5 (Pin_5); no longer U7.23 (SEG_D)
- net C55: now also U7.20 (SEG_C), J10.4 (Pin_4); no longer U7.21 (SEG_E)
- net C56: now also U7.21 (SEG_E), J10.3 (Pin_3); no longer U7.15 (SEG_F)
- net C57: now also U7.22 (SEG_DP), J10.2 (Pin_2); no longer U7.17 (SEG_G)
- net C58: now also U7.23 (SEG_D), J10.1 (Pin_1); no longer U7.22 (SEG_DP)
- net C61: now also J15.8 (Pin_8)
- net C62: now also U8.15 (SEG_F), J15.7 (Pin_7); no longer U8.16 (SEG_B)
- net C63: now also U8.16 (SEG_B), J15.6 (Pin_6); no longer U8.20 (SEG_C)
- net C64: now also U8.17 (SEG_G), J15.5 (Pin_5); no longer U8.23 (SEG_D)
- net C65: now also U8.20 (SEG_C), J14.4 (Pin_4); no longer U8.21 (SEG_E)
- net C66: now also U8.21 (SEG_E), J14.3 (Pin_3); no longer U8.15 (SEG_F)
- net C67: now also U8.22 (SEG_DP), J14.2 (Pin_2); no longer U8.17 (SEG_G)
- net C68: now also U8.23 (SEG_D), J14.1 (Pin_1); no longer U8.22 (SEG_DP)
- net C71: now also J13.8 (Pin_8)
- net C72: now also U9.15 (SEG_F), J13.7 (Pin_7); no longer U9.16 (SEG_B)
- net C73: now also U9.16 (SEG_B), J13.6 (Pin_6); no longer U9.20 (SEG_C)
- net C74: now also U9.17 (SEG_G), J13.5 (Pin_5); no longer U9.23 (SEG_D)
- net C75: now also U9.20 (SEG_C), J12.4 (Pin_4); no longer U9.21 (SEG_E)
- net C76: now also U9.21 (SEG_E), J12.3 (Pin_3); no longer U9.15 (SEG_F)
- net C77: now also U9.22 (SEG_DP), J12.2 (Pin_2); no longer U9.17 (SEG_G)
- net C78: now also U9.23 (SEG_D), J12.1 (Pin_1); no longer U9.22 (SEG_DP)
- net C81: now also J17.8 (Pin_8)
- net C82: now also U10.15 (SEG_F), J17.7 (Pin_7); no longer U10.16 (SEG_B)
- net C83: now also U10.16 (SEG_B), J17.6 (Pin_6); no longer U10.20 (SEG_C)
- net C84: now also U10.17 (SEG_G), J17.5 (Pin_5); no longer U10.23 (SEG_D)
- net C85: now also U10.20 (SEG_C), J16.4 (Pin_4); no longer U10.21 (SEG_E)
- net C86: now also U10.21 (SEG_E), J16.3 (Pin_3); no longer U10.15 (SEG_F)
- net C87: now also U10.22 (SEG_DP), J16.2 (Pin_2); no longer U10.17 (SEG_G)
- net C88: now also U10.23 (SEG_D), J16.1 (Pin_1); no longer U10.22 (SEG_DP)
- net R51: now also J10.8 (Pin_8)
- net R52: now also U7.3 (DIG_4), J10.7 (Pin_7); no longer U7.11 (DIG_1)
- net R53: now also U7.5 (DIG_6), J10.6 (Pin_6); no longer U7.6 (DIG_2)
- net R54: now also U7.6 (DIG_2), J10.5 (Pin_5); no longer U7.7 (DIG_3)
- net R55: now also U7.7 (DIG_3), J11.4 (Pin_4); no longer U7.3 (DIG_4)
- net R56: now also U7.8 (DIG_7), J11.3 (Pin_3); no longer U7.10 (DIG_5)
- net R57: now also U7.10 (DIG_5), J11.2 (Pin_2); no longer U7.5 (DIG_6)
- net R58: now also U7.11 (DIG_1), J11.1 (Pin_1); no longer U7.8 (DIG_7)
- net R61: now also J14.8 (Pin_8)
- net R62: now also U8.3 (DIG_4), J14.7 (Pin_7); no longer U8.11 (DIG_1)
- net R63: now also U8.5 (DIG_6), J14.6 (Pin_6); no longer U8.6 (DIG_2)
- net R64: now also U8.6 (DIG_2), J14.5 (Pin_5); no longer U8.7 (DIG_3)
- net R65: now also U8.7 (DIG_3), J15.4 (Pin_4); no longer U8.3 (DIG_4)
- net R66: now also U8.8 (DIG_7), J15.3 (Pin_3); no longer U8.10 (DIG_5)
- net R67: now also U8.10 (DIG_5), J15.2 (Pin_2); no longer U8.5 (DIG_6)
- net R68: now also U8.11 (DIG_1), J15.1 (Pin_1); no longer U8.8 (DIG_7)
- net R71: now also J12.8 (Pin_8)
- net R72: now also U9.3 (DIG_4), J12.7 (Pin_7); no longer U9.11 (DIG_1)
- net R73: now also U9.5 (DIG_6), J12.6 (Pin_6); no longer U9.6 (DIG_2)
- net R74: now also U9.6 (DIG_2), J12.5 (Pin_5); no longer U9.7 (DIG_3)
- net R75: now also U9.7 (DIG_3), J13.4 (Pin_4); no longer U9.3 (DIG_4)
- net R76: now also U9.8 (DIG_7), J13.3 (Pin_3); no longer U9.10 (DIG_5)
- net R77: now also U9.10 (DIG_5), J13.2 (Pin_2); no longer U9.5 (DIG_6)
- net R78: now also U9.11 (DIG_1), J13.1 (Pin_1); no longer U9.8 (DIG_7)
- net R81: now also J16.8 (Pin_8)
- net R82: now also U10.3 (DIG_4), J16.7 (Pin_7); no longer U10.11 (DIG_1)
- net R83: now also U10.5 (DIG_6), J16.6 (Pin_6); no longer U10.6 (DIG_2)
- net R84: now also U10.6 (DIG_2), J16.5 (Pin_5); no longer U10.7 (DIG_3)
- net R85: now also U10.7 (DIG_3), J17.4 (Pin_4); no longer U10.3 (DIG_4)
- net R86: now also U10.8 (DIG_7), J17.3 (Pin_3); no longer U10.10 (DIG_5)
- net R87: now also U10.10 (DIG_5), J17.2 (Pin_2); no longer U10.5 (DIG_6)
- net R88: now also U10.11 (DIG_1), J17.1 (Pin_1); no longer U10.8 (DIG_7)
