File: PCB Class/esp32.kicad_sch (KiCad schematic)
At the start: 1 part, among them U1 ESP32-S3-WROOM-1-N4

Commit message: Final Schematic
Parts:
- added C12: 1uF, symbol Device:C_Small
- added C9: 100nF, Capacitor_SMD:C_0402_1005Metric, symbol Device:C_Small
- added R7: 10K, Resistor_SMD:R_0402_1005Metric, symbol Device:R_Small
- added SW1: SW_Push, symbol Switch:SW_Push
Connections:
- net +3.3V: now also C12.1, R7.1
- net DIN1: now also U1.22 (IO14); no longer U1.38 (IO2)
- net DIN2: now also U1.9 (IO16); no longer U1.4 (IO4)
- net DIN3: now also U1.38 (IO2); no longer U1.6 (IO6)
- net DIN4: now also U1.4 (IO4); no longer U1.12 (IO8)
- net GND: now also C12.2, C9.2, SW1.1
- net LOAD1: now also U1.21 (IO13); no longer U1.39 (IO1)
- net LOAD2: now also U1.8 (IO15); no longer U1.15 (IO3)
- net LOAD3: now also U1.39 (IO1); no longer U1.5 (IO5)
- net LOAD4: now also U1.15 (IO3); no longer U1.7 (IO7)
- net LOAD7: now reaches U1.10 (IO17)
- net DIN7: now reaches U1.11 (IO18)
- net at U1.27 (IO0): now also SW1.2
- net LOAD8: now reaches U1.28 (IO35)
- net RST: now reaches U1.3 (EN)
- net RST: now also C9.1, R7.2
- net CLK1 renamed CLK
- net CLK2: no longer names the net of U1.33 (IO40)
- net CLK3: no longer names the net of U1.34 (IO41)
- net CLK4 renamed DIN8
- new net DIN5: U1.6 (IO6)
- new net DIN6: U1.12 (IO8)
- new net LOAD5: U1.5 (IO5)
- new net LOAD6: U1.7 (IO7)
- no-connect marks 23 -> 16
Other:
- note removed: "Jan 10th 2024"
- note removed: "Riya Gupta LED Light Schematic"
- title: (none) -> RGB LED Lights

Commit message: Footprints
Parts:
- C1: renamed from C12; footprint (none) -> Capacitor_SMD:C_0603_1608Metric
- C2: renamed from C9; footprint Capacitor_SMD:C_0402_1005Metric -> Capacitor_SMD:C_0603_1608Metric
- R3: renamed from R7; footprint Resistor_SMD:R_0402_1005Metric -> Resistor_SMD:R_0603_1608Metric
- SW1: footprint (none) -> Button_Switch_SMD:SW_SPST_FSMSM
Changed lines of the file:
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@@
       (effects (font (size 1.27 1.27)) (justify right))
     )
-    (property "Footprint" "" (id 2) (at 105.41 67.31 0)
+    (property "Footprint" "Button_Switch_SMD:SW_SPST_FSMSM" (id 2) (at 105.41 67.31 0)
       (effects (font (size 1.27 1.27)) hide)
     )
@@
   (symbol (lib_id "Device:R_Small") (at 115.57 43.18 0) (unit 1)
     (in_bom yes) (on_board yes) (fields_autoplaced)
-    (property "Reference" "R7" (id 0) (at 118.11 41.9099 0)
+    (property "Reference" "R3" (id 0) (at 118.11 41.9099 0)
       (effects (font (size 1.27 1.27)) (justify left))
     )
@@
       (effects (font (size 1.27 1.27)) (justify left))
     )
-    (property "Footprint" "Resistor_SMD:R_0402_1005Metric" (id 2) (at 115.57 43.18 0)
+    (property "Footprint" "Resistor_SMD:R_0603_1608Metric" (id 2) (at 115.57 43.18 0)
       (effects (font (size 1.27 1.27)) hide)
     )
@@
   (symbol (lib_id "Device:C_Small") (at 115.57 50.8 0) (unit 1)
     (in_bom yes) (on_board yes) (fields_autoplaced)
-    (property "Reference" "C9" (id 0) (at 118.11 49.5362 0)
+    (property "Reference" "C2" (id 0) (at 118.11 49.5362 0)
       (effects (font (size 1.27 1.27)) (justify left))
     )
@@
       (effects (font (size 1.27 1.27)) (justify left))
     )
-    (property "Footprint" "Capacitor_SMD:C_0402_1005Metric" (id 2) (at 115.57 50.8 0)
+    (property "Footprint" "Capacitor_SMD:C_0603_1608Metric" (id 2) (at 115.57 50.8 0)
       (effects (font (size 1.27 1.27)) hide)
     )
@@
   (symbol (lib_id "Device:C_Small") (at 160.02 49.53 0) (unit 1)
     (in_bom yes) (on_board yes) (fields_autoplaced)
-    (property "Reference" "C12" (id 0) (at 162.56 48.2662 0)
+    (property "Reference" "C1" (id 0) (at 162.56 48.2662 0)
       (effects (font (size 1.27 1.27)) (justify left))
     )
@@
       (effects (font (size 1.27 1.27)) (justify left))
     )
-    (property "Footprint" "" (id 2) (at 160.02 49.53 0)
+    (property "Footprint" "Capacitor_SMD:C_0603_1608Metric" (id 2) (at 160.02 49.53 0)
       (effects (font (size 1.27 1.27)) hide)
     )

Commit message: Layout
Parts:
- removed C2: 100nF, Capacitor_SMD:C_0603_1608Metric, symbol Device:C_Small
- U1: footprint ESP32-S3-WROOM-1-N4:XCVR_ESP32-S3-WROOM-1-N4 -> ESP32_S3_WROOM_1_N4 (1):XCVR_ESP32-S3-WROOM-1-N4
- renumbered R3 to R11
Connections:
- net CLK: now also U1.20 (IO12); no longer U1.32 (IO39)
- net DIN1: now also U1.5 (IO5); no longer U1.22 (IO14)
- net DIN3: now also U1.22 (IO14); no longer U1.38 (IO2)
- net DIN4: now also U1.29 (IO36); no longer U1.4 (IO4)
- net DIN5: now also U1.7 (IO7); no longer U1.6 (IO6)
- net DIN6: now also U1.17 (IO9); no longer U1.12 (IO8)
- net DIN7: now also U1.19 (IO11); no longer U1.11 (IO18)
- net DIN8: now also U1.24 (IO47); no longer U1.29 (IO36)
- net LOAD1: now also U1.4 (IO4); no longer U1.21 (IO13)
- net LOAD3: now also U1.21 (IO13); no longer U1.39 (IO1)
- net LOAD4: now also U1.28 (IO35); no longer U1.15 (IO3)
- net LOAD5: now also U1.6 (IO6); no longer U1.5 (IO5)
- net LOAD6: now also U1.16 (IO46); no longer U1.7 (IO7)
- net LOAD7: now also U1.18 (IO10); no longer U1.10 (IO17)
- net LOAD8: now also U1.23 (IO21); no longer U1.28 (IO35)
- net RST: now also SW1.2
- net at U1.27 (IO0): no longer SW1.2
- no-connect marks 16 -> 17
Other:
- moved on the sheet: SW1

Commit message: Final Layout
Parts:
- added SW2: SW_Push, Button_Switch_SMD:SW_SPST_FSMSM, symbol Switch:SW_Push
Connections:
- net CLK: now also U1.18 (IO10); no longer U1.20 (IO12)
- net DIN1: now also U1.7 (IO7); no longer U1.5 (IO5)
- net DIN2: now also U1.17 (IO9); no longer U1.9 (IO16)
- net DIN5: now also U1.5 (IO5); no longer U1.7 (IO7)
- net DIN6: now also U1.9 (IO16); no longer U1.17 (IO9)
- net DIN7: now also U1.20 (IO12); no longer U1.19 (IO11)
- net GND: now also SW2.1
- net LOAD1: now also U1.6 (IO6); no longer U1.4 (IO4)
- net LOAD2: now also U1.16 (IO46); no longer U1.8 (IO15)
- net LOAD5: now also U1.4 (IO4); no longer U1.6 (IO6)
- net LOAD6: now also U1.8 (IO15); no longer U1.16 (IO46)
- net LOAD7: now also U1.19 (IO11); no longer U1.18 (IO10)
- net at U1.27 (IO0): now also SW2.2
- no-connect marks 17 -> 16
Other:
- moved on the sheet: SW1
