File: PCB Class/leds.kicad_sch (KiCad schematic)
At the start: 100 parts

Commit message: Final Schematic
Parts:
- removed D? (x36): LED, symbol Device:LED
- gave numbers to parts that had none: 64
Connections:
- net C1 1-8 renamed C11
- net C2 1-8 renamed C12
- net C3 1-8 renamed C13
- net C4 1-8 renamed C14
- net C5 1-8 renamed C15
- net C6 1-8 renamed C16
- net C7 1-8 renamed C17
- net C8 1-8 renamed C18
- net R1 1-8 renamed R11
- net R2 1-8 renamed R12
- net R3 1-8 renamed R13
- net R4 1-8 renamed R14
- net R5 1-8 renamed R15
- net R6 1-8 renamed R16
- net R7 1-8 renamed R17
- net R8 1-8 renamed R18
Other:
- note added: "This is what one of the LED panels will look like. I'm planning on stacking 8 to make a cube. These LEDs will not be on the PCB, but it is here to show how it connects."
- title: (none) -> RGB LED Lights
- moved on the sheet: D1, D11, D12, D13, D14, D15, D16, D17, D18, D2, D21, D22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

Commit message: Footprints
Parts:
- D1, D11, D12, D13, D14, D15, D2, D3, D4, D5, D6, D7, D8: footprint (none) -> LED_SMD:LED_0201_0603Metric
