File: PCB Class/usbc.kicad_sch (KiCad schematic)
At the start: 3 parts

Commit message: Final Schematic
Parts:
- gave numbers to parts that had none: 3
Connections:
- net CC1: now also R2.1; no longer R2.2
- net CC2: now also R1.1; no longer R1.2
- net GND: now also R1.2, R2.2; no longer R1.1, R2.1
Other:
- note removed: "Jan 10th 2024"
- note removed: "Riya Gupta LED Light Schematic"
- title: (none) -> RGB LED Lights
- moved on the sheet: R1, R2
Changed lines of the file:
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@@
 (kicad_sch (version 20211123) (generator eeschema)
-  (paper "A4")
+  (paper "USLetter")
+  (title_block
+    (title "RGB LED Lights")
+    (date "2024-01-11")
+    (rev "B01")
+    (comment 1 "Riya Gupta")
+  )
   (junction (at 144.78 83.82) (diameter 0) (color 0 0 0 0)
   )
@@
   (no_connect (at 144.78 99.06))
   (no_connect (at 144.78 96.52))
-  (wire (pts (xy 162.56 73.66) (xy 162.56 76.2))
+  (wire (pts (xy 144.78 73.66) (xy 168.91 73.66))
     (stroke (width 0) (type default) (color 0 0 0 0))
   )
-  (wire (pts (xy 162.56 64.77) (xy 162.56 66.04))
+  (wire (pts (xy 158.75 86.36) (xy 158.75 85.09))
     (stroke (width 0) (type default) (color 0 0 0 0))
   )
@@
     (stroke (width 0) (type default) (color 0 0 0 0))
   )
-  (wire (pts (xy 162.56 76.2) (xy 144.78 76.2))
+  (wire (pts (xy 158.75 76.2) (xy 144.78 76.2))
     (stroke (width 0) (type default) (color 0 0 0 0))
   )
   (wire (pts (xy 121.92 106.68) (xy 129.54 106.68))
+    (stroke (width 0) (type default) (color 0 0 0 0))
+  )
+  (wire (pts (xy 168.91 73.66) (xy 168.91 76.2))
     (stroke (width 0) (type default) (color 0 0 0 0))
   )
@@
     (stroke (width 0) (type default) (color 0 0 0 0))
   )
-  (wire (pts (xy 152.4 73.66) (xy 144.78 73.66))
+  (wire (pts (xy 158.75 76.2) (xy 158.75 77.47))
     (stroke (width 0) (type default) (color 0 0 0 0))
   )
-  (wire (pts (xy 152.4 64.77) (xy 152.4 66.04))
+  (wire (pts (xy 168.91 83.82) (xy 168.91 86.36))
     (stroke (width 0) (type default) (color 0 0 0 0))
-  )
-  (text "Riya Gupta LED Light Schematic" (at 187.96 190.5 0)
-    (effects (font (size 1.27 1.27)) (justify left bottom))
-  )
-  (text "Jan 10th 2024" (at 207.01 194.31 0)
-    (effects (font (size 1.27 1.27)) (justify left bottom))
   )
   (label "CC2" (at 144.78 76.2 0)
@@
     (effects (font (size 1.27 1.27)) (justify left bottom))
   )
-  (hierarchical_label "D-" (shape bidirectional) (at 147.32 83.82 0)
+  (hierarchical_label "D+" (shape output) (at 147.32 88.9 0)
     (effects (font (size 1.27 1.27)) (justify left))
   )
-  (hierarchical_label "D+" (shape bidirectional) (at 147.32 88.9 0)
+  (hierarchical_label "D-" (shape output) (at 147.32 83.82 0)
     (effects (font (size 1.27 1.27)) (justify left))
   )
   (symbol (lib_id "power:+5V") (at 144.78 68.58 0) (unit 1)
     (in_bom yes) (on_board yes) (fields_autoplaced)
-    (property "Reference" "#PWR?" (id 0) (at 144.78 72.39 0)
+    (property "Reference" "#PWR0105" (id 0) (at 144.78 72.39 0)
       (effects (font (size 1.27 1.27)) hide)
     )
@@
   (symbol (lib_id "Connector:USB_C_Receptacle_USB2.0") (at 129.54 83.82 0) (unit 1)
     (in_bom yes) (on_board yes) (fields_autoplaced)
-    (property "Reference" "J?" (id 0) (at 129.54 60.96 0))
+    (property "Reference" "J1" (id 0) (at 129.54 60.96 0))
     (property "Value" "USB_C_Receptacle_USB2.0" (id 1) (at 129.54 63.5 0))
     (property "Footprint" "" (id 2) (at 133.35 83.82 0)
@@
     (pin "S1")
   )
-  (symbol (lib_id "power:GND") (at 152.4 64.77 180) (unit 1)
+  (symbol (lib_id "power:GND") (at 168.91 86.36 0) (unit 1)
     (in_bom yes) (on_board yes) (fields_autoplaced)
-    (property "Reference" "#PWR?" (id 0) (at 152.4 58.42 0)
+    (property "Reference" "#PWR0104" (id 0) (at 168.91 92.71 0)
       (effects (font (size 1.27 1.27)) hide)
     )
-    (property "Value" "GND" (id 1) (at 152.4 59.69 0))
-    (property "Footprint" "" (id 2) (at 152.4 64.77 0)
+    (property "Value" "GND" (id 1) (at 168.91 91.44 0))
+    (property "Footprint" "" (id 2) (at 168.91 86.36 0)
       (effects (font (size 1.27 1.27)) hide)
     )
-    (property "Datasheet" "" (id 3) (at 152.4 64.77 0)
+    (property "Datasheet" "" (id 3) (at 168.91 86.36 0)
       (effects (font (size 1.27 1.27)) hide)
     )
     (pin "1")
   )
-  (symbol (lib_id "Device:R") (at 162.56 69.85 0) (unit 1)
+  (symbol (lib_id "Device:R") (at 158.75 81.28 0) (unit 1)
     (in_bom yes) (on_board yes) (fields_autoplaced)
-    (property "Reference" "R?" (id 0) (at 165.1 68.5799 0)
+    (property "Reference" "R1" (id 0) (at 161.29 80.0099 0)
       (effects (font (size 1.27 1.27)) (justify left))
     )
-    (property "Value" "5.1K" (id 1) (at 165.1 71.1199 0)
+    (property "Value" "5.1K" (id 1) (at 161.29 82.5499 0)
       (effects (font (size 1.27 1.27)) (justify left))
     )
-    (property "Footprint" "" (id 2) (at 160.782 69.85 90)
+    (property "Footprint" "" (id 2) (at 156.972 81.28 90)
       (effects (font (size 1.27 1.27)) hide)
     )
-    (property "Datasheet" "~" (id 3) (at 162.56 69.85 0)
+    (property "Datasheet" "~" (id 3) (at 158.75 81.28 0)
       (effects (font (size 1.27 1.27)) hide)
     )
@@
     (pin "2")
   )
-  (symbol (lib_id "power:GND") (at 162.56 64.77 180) (unit 1)
+  (symbol (lib_id "power:GND") (at 158.75 86.36 0) (unit 1)
     (in_bom yes) (on_board yes) (fields_autoplaced)
-    (property "Reference" "#PWR?" (id 0) (at 162.56 58.42 0)
+    (property "Reference" "#PWR0103" (id 0) (at 158.75 92.71 0)
       (effects (font (size 1.27 1.27)) hide)
     )
-    (property "Value" "GND" (id 1) (at 162.56 59.69 0))
-    (property "Footprint" "" (id 2) (at 162.56 64.77 0)
+    (property "Value" "GND" (id 1) (at 158.75 91.44 0))
+    (property "Footprint" "" (id 2) (at 158.75 86.36 0)
       (effects (font (size 1.27 1.27)) hide)
     )
-    (property "Datasheet" "" (id 3) (at 162.56 64.77 0)
+    (property "Datasheet" "" (id 3) (at 158.75 86.36 0)
       (effects (font (size 1.27 1.27)) hide)
     )
@@
   (symbol (lib_id "power:GND") (at 129.54 106.68 0) (unit 1)
     (in_bom yes) (on_board yes) (fields_autoplaced)
-    (property "Reference" "#PWR?" (id 0) (at 129.54 113.03 0)
+    (property "Reference" "#PWR0102" (id 0) (at 129.54 113.03 0)
       (effects (font (size 1.27 1.27)) hide)
     )
@@
     (pin "1")
   )
-  (symbol (lib_id "Device:R") (at 152.4 69.85 0) (unit 1)
+  (symbol (lib_id "Device:R") (at 168.91 80.01 0) (unit 1)
     (in_bom yes) (on_board yes) (fields_autoplaced)
-    (property "Reference" "R?" (id 0) (at 154.94 68.5799 0)
+    (property "Reference" "R2" (id 0) (at 171.45 78.7399 0)
       (effects (font (size 1.27 1.27)) (justify left))
     )
-    (property "Value" "5.1K" (id 1) (at 154.94 71.1199 0)
+    (property "Value" "5.1K" (id 1) (at 171.45 81.2799 0)
       (effects (font (size 1.27 1.27)) (justify left))
     )
-    (property "Footprint" "" (id 2) (at 150.622 69.85 90)
+    (property "Footprint" "" (id 2) (at 167.132 80.01 90)
       (effects (font (size 1.27 1.27)) hide)
     )
-    (property "Datasheet" "~" (id 3) (at 152.4 69.85 0)
+    (property "Datasheet" "~" (id 3) (at 168.91 80.01 0)
       (effects (font (size 1.27 1.27)) hide)
     )

Commit message: Footprints
Parts:
- J1: footprint (none) -> Connector_USB:USB_C_Receptacle_GCT_USB4085
- R1, R2: footprint (none) -> Resistor_SMD:R_0603_1608Metric
Changed lines of the file:
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@@
     (property "Reference" "J1" (id 0) (at 129.54 60.96 0))
     (property "Value" "USB_C_Receptacle_USB2.0" (id 1) (at 129.54 63.5 0))
-    (property "Footprint" "" (id 2) (at 133.35 83.82 0)
+    (property "Footprint" "Connector_USB:USB_C_Receptacle_GCT_USB4085" (id 2) (at 133.35 83.82 0)
       (effects (font (size 1.27 1.27)) hide)
     )
@@
       (effects (font (size 1.27 1.27)) (justify left))
     )
-    (property "Footprint" "" (id 2) (at 156.972 81.28 90)
+    (property "Footprint" "Resistor_SMD:R_0603_1608Metric" (id 2) (at 156.972 81.28 90)
       (effects (font (size 1.27 1.27)) hide)
     )
@@
       (effects (font (size 1.27 1.27)) (justify left))
     )
-    (property "Footprint" "" (id 2) (at 167.132 80.01 90)
+    (property "Footprint" "Resistor_SMD:R_0603_1608Metric" (id 2) (at 167.132 80.01 90)
       (effects (font (size 1.27 1.27)) hide)
     )
